Commit message: Clean up

File: pcr_description/urdf/pcr_workcell.urdf (robot description, URDF)
Before this commit: robot PCR Workcell, 48 links, 47 joints
Joints:
- joint Biometra_Base: child biometra/biometra_base -> biometra_base; parent module_carts/cart_2 -> cart_2
- joint Biometra_Base2: child biometra/biometra_base2 -> biometra_base2; parent module_carts/cart_2 -> cart_2
- joint Hidex_Base: child hidex/hidex_body -> hidex_body; parent module_carts/cart_3 -> cart_3
- joint OT2_alpha: child ot2/OT2_alpha -> OT2_alpha; parent module_carts/cart_8 -> cart_8
- joint OT2_betha: child ot2/OT2_betha -> OT2_betha; parent module_carts/cart_7 -> cart_7
- joint OT2_gamma: child ot2/OT2_gamma -> OT2_gamma; parent module_carts/cart_4 -> cart_4
- joint Peeler_Base: child peeler/peeler_base -> peeler_base; parent module_carts/cart_6 -> cart_6
- joint Sciclops_Base: child sciclops/sciclops_base -> sciclops_base; parent module_carts/cart_5 -> cart_5
- joint Sealer_Base: child sealer/sealer_base -> sealer_base; parent module_carts/cart_6 -> cart_6
- joint pf400_module: child pf400/rail_base -> rail_base; parent module_carts/pf400_cart -> pf400_cart
