Commit message: Changing module import name

File: pcr_description/urdf/pcr_workcell.urdf.xacro (robot description, xacro)
@@ -15,7 +15,7 @@
   <xacro:include filename="$(find ot2_description)/urdf/OT2.urdf.xacro" />
   <xacro:OT2 prefix="ot2/"/>
-  <!-- Thermocycler -->
-  <xacro:include filename="$(find biometra_description)/urdf/thermocycler.urdf.xacro" />
-  <xacro:Thermocycler prefix="thermocycler/"/>
+  <!-- Biometra -->
+  <xacro:include filename="$(find biometra_description)/urdf/biometra.urdf.xacro" />
+  <xacro:Biometra prefix="biometra/"/>
   <!-- Hidex -->
   <xacro:include filename="$(find hidex_description)/urdf/hidex.urdf.xacro" />
@@ -32,14 +32,14 @@
     <limit effort="1000.0" lower="0" upper="0" velocity="0.5"/>
   </joint>
-  <joint name="Thermocycler_Base" type="fixed">
+  <joint name="Biometra_Base" type="fixed">
     <parent link="module_carts/cart_2"/>
-    <child link="thermocycler/thermocycler_base"/>
+    <child link="biometra/biometra_base"/>
     <axis xyz="0 0 0"/>
     <origin xyz="0.2 -0.62 0" rpy="0 0 0"/>
     <limit effort="1000.0" lower="0" upper="0" velocity="0.5"/>
   </joint>
-  <joint name="Thermocycler_Base2" type="fixed">
+  <joint name="Biometra_Base2" type="fixed">
     <parent link="module_carts/cart_2"/>
-    <child link="thermocycler/thermocycler_base2"/>
+    <child link="biometra/biometra_base2"/>
     <axis xyz="0 0 0"/>
     <origin xyz="-0.1 -0.62 0" rpy="0 0 0"/>

Commit message: Adding sciclops description

File: pcr_description/urdf/pcr_workcell.urdf.xacro (robot description, xacro)
@@ -24,4 +24,7 @@
   <xacro:include filename="$(find pcr_description)/urdf/module_carts.urdf.xacro" />
   <xacro:Module_Carts prefix="module_carts/"/>
+  <!-- Sciclops -->
+  <xacro:include filename="$(find sciclops_description)/urdf/sciclops.urdf.xacro" />
+  <xacro:Sciclops prefix="sciclops/"/>
   <!-- Wrokcell Setup -->
   <joint name="pf400_module" type="fixed">
@@ -29,5 +32,5 @@
     <child link="pf400/rail_base"/>
     <axis xyz="0 0 0"/>
-    <origin xyz="-0.14 -0.0198 0.835" rpy="0 0 0"/>
+    <origin xyz="-0.14 -0.0198 0.83" rpy="0 0 0"/>
     <limit effort="1000.0" lower="0" upper="0" velocity="0.5"/>
   </joint>
@@ -36,5 +39,5 @@
     <child link="biometra/biometra_base"/>
     <axis xyz="0 0 0"/>
-    <origin xyz="0.2 -0.62 0" rpy="0 0 0"/>
+    <origin xyz="0.2 -0.62 0.01" rpy="0 0 0"/>
     <limit effort="1000.0" lower="0" upper="0" velocity="0.5"/>
   </joint>
@@ -43,5 +46,12 @@
     <child link="biometra/biometra_base2"/>
     <axis xyz="0 0 0"/>
-    <origin xyz="-0.1 -0.62 0" rpy="0 0 0"/>
+    <origin xyz="-0.1 -0.62 0.01" rpy="0 0 0"/>
+    <limit effort="1000.0" lower="0" upper="0" velocity="0.5"/>
+  </joint>
+ <joint name="Sciclops_Base" type="fixed">
+    <parent link="module_carts/cart_5"/>
+    <child link="sciclops/sciclops_base"/>
+    <axis xyz="0 0 0"/>
+    <origin xyz="0 -0.04 1.05" rpy="0 0 5.1"/>
     <limit effort="1000.0" lower="0" upper="0" velocity="0.5"/>
   </joint>
@@ -50,5 +60,5 @@
     <child link="peeler/peeler_base"/>
     <axis xyz="0 0 0"/>
-    <origin xyz="-0.13 0.15 1.042" rpy="0 0 0"/>
+    <origin xyz="-0.13 0.15 1.052" rpy="0 0 0"/>
     <limit effort="1000.0" lower="0" upper="0" velocity="0.5"/>
   </joint>
@@ -57,5 +67,5 @@
     <child link="sealer/sealer_base"/>
     <axis xyz="0 0 0"/>
-    <origin xyz="0.27 -0.53 1.042" rpy="0 0 0"/>
+    <origin xyz="0.27 -0.53 1.052" rpy="0 0 0"/>
     <limit effort="1000.0" lower="0" upper="0" velocity="0.5"/>
   </joint>
@@ -64,5 +74,5 @@
     <child link="hidex/hidex_body"/>
     <axis xyz="0 0 0"/>
-    <origin xyz="0.2 -0.45 1.042" rpy="0 0 0"/>
+    <origin xyz="0.2 -0.45 1.052" rpy="0 0 0"/>
     <limit effort="1000.0" lower="0" upper="0" velocity="0.5"/>
   </joint>
@@ -71,5 +81,5 @@
     <child link="ot2/OT2_alpha"/>
     <axis xyz="0 0 0"/>
-    <origin xyz="0.825 0.47 0" rpy="0 0 3.1416"/>
+    <origin xyz="0.825 0.47 0.01" rpy="0 0 3.1416"/>
     <limit effort="1000.0" lower="0" upper="0" velocity="0.5"/>
   </joint>
@@ -78,5 +88,12 @@
     <child link="ot2/OT2_betha"/>
     <axis xyz="0 0 0"/>
-    <origin xyz="0.825 0.47 0" rpy="0 0 3.1416"/>
+    <origin xyz="0.825 0.47 0.01" rpy="0 0 3.1416"/>
+    <limit effort="1000.0" lower="0" upper="0" velocity="0.5"/>
+  </joint>
+  <joint name="OT2_gamma" type="fixed">
+    <parent link="module_carts/cart_4"/>
+    <child link="ot2/OT2_gamma"/>
+    <axis xyz="0 0 0"/>
+    <origin xyz="-0.52 -0.85 0.01" rpy="0 0 0"/>
     <limit effort="1000.0" lower="0" upper="0" velocity="0.5"/>
   </joint>

Commit message: Adding plate exchange deck

File: pcr_description/urdf/pcr_workcell.urdf.xacro (robot description, xacro)
@@ -27,4 +27,7 @@
   <xacro:include filename="$(find sciclops_description)/urdf/sciclops.urdf.xacro" />
   <xacro:Sciclops prefix="sciclops/"/>
+  <!-- Plate Exchange Deck -->
+  <xacro:include filename="$(find sciclops_description)/urdf/plate_exchange.xacro" />
+  <xacro:plate_exchange_deck prefix="exchange_deck/"/>
   <!-- Wrokcell Setup -->
   <joint name="pf400_module" type="fixed">
@@ -98,3 +101,10 @@
     <limit effort="1000.0" lower="0" upper="0" velocity="0.5"/>
   </joint>
+  <joint name="Exchange_Deck_Base" type="fixed">
+    <parent link="module_carts/cart_1"/>
+    <child link="exchange_deck/plate_exchange"/>
+    <axis xyz="0 0 0"/>
+    <origin xyz="-0.09 -0.4 1.05" rpy="0 0 1.6"/>
+    <limit effort="1000.0" lower="0" upper="0" velocity="0.5"/>
+  </joint>
 </robot>

Commit message: Module location update

File: pcr_description/urdf/pcr_workcell.urdf.xacro (robot description, xacro)
@@ -105,5 +105,5 @@
     <child link="exchange_deck/plate_exchange"/>
     <axis xyz="0 0 0"/>
-    <origin xyz="-0.09 -0.4 1.05" rpy="0 0 1.6"/>
+    <origin xyz="-0.078 -0.4 1.058" rpy="0 0 1.6"/>
     <limit effort="1000.0" lower="0" upper="0" velocity="0.5"/>
   </joint>
