Commit message: Edditing module cart locations

File: pcr_description/urdf/module_carts.urdf.xacro (robot description, xacro)
@@ -7,5 +7,5 @@
       <origin xyz="0 0 0" rpy="0 0 0"/>
       <geometry>
-        <mesh filename="package://pf400_description/meshes/module_cart.stl" scale="1 1 1"/>
+        <mesh filename="package://pcr_description/meshes/module_cart.stl" scale="1 1 1"/>
       </geometry>
       <material name="darkbluegreen"/>
@@ -13,5 +13,5 @@
     <collision>
       <geometry>
-        <mesh filename="package://pf400_description/meshes/module_cart.stl" scale="1 1 1"/>
+        <mesh filename="package://pcr_description/meshes/module_cart.stl" scale="1 1 1"/>
       </geometry>
       <origin xyz="0 0 0" rpy="0 0 0"/>
@@ -22,5 +22,5 @@
       <origin xyz="0 0 0" rpy="0 0 0"/>
       <geometry>
-        <mesh filename="package://pf400_description/meshes/module_cart.stl" scale="1 1 1"/>
+        <mesh filename="package://pcr_description/meshes/module_cart.stl" scale="1 1 1"/>
       </geometry>
       <material name="darkbluegreen"/>
@@ -28,5 +28,5 @@
     <collision>
       <geometry>
-        <mesh filename="package://pf400_description/meshes/module_cart.stl" scale="1 1 1"/>
+        <mesh filename="package://pcr_description/meshes/module_cart.stl" scale="1 1 1"/>
       </geometry>
       <origin xyz="0 0 0" rpy="0 0 0"/>
@@ -37,5 +37,5 @@
       <origin xyz="0 0 0" rpy="0 0 0"/>
       <geometry>
-        <mesh filename="package://pf400_description/meshes/module_cart.stl" scale="1 1 1"/>
+        <mesh filename="package://pcr_description/meshes/module_cart.stl" scale="1 1 1"/>
       </geometry>
       <material name="darkbluegreen"/>
@@ -43,5 +43,5 @@
     <collision>
       <geometry>
-        <mesh filename="package://pf400_description/meshes/module_cart.stl" scale="1 1 1"/>
+        <mesh filename="package://pcr_description/meshes/module_cart.stl" scale="1 1 1"/>
       </geometry>
       <origin xyz="0 0 0" rpy="0 0 0"/>
@@ -52,5 +52,5 @@
       <origin xyz="0 0 0" rpy="0 0 0"/>
       <geometry>
-        <mesh filename="package://pf400_description/meshes/module_cart.stl" scale="1 1 1"/>
+        <mesh filename="package://pcr_description/meshes/module_cart.stl" scale="1 1 1"/>
       </geometry>
       <material name="darkbluegreen"/>
@@ -58,5 +58,5 @@
     <collision>
       <geometry>
-        <mesh filename="package://pf400_description/meshes/module_cart.stl" scale="1 1 1"/>
+        <mesh filename="package://pcr_description/meshes/module_cart.stl" scale="1 1 1"/>
       </geometry>
       <origin xyz="0 0 0" rpy="0 0 0"/>
@@ -67,5 +67,5 @@
       <origin xyz="0 0 0" rpy="0 0 0"/>
       <geometry>
-        <mesh filename="package://pf400_description/meshes/module_cart.stl" scale="1 1 1"/>
+        <mesh filename="package://pcr_description/meshes/module_cart.stl" scale="1 1 1"/>
       </geometry>
       <material name="darkbluegreen"/>
@@ -73,5 +73,5 @@
     <collision>
       <geometry>
-        <mesh filename="package://pf400_description/meshes/module_cart.stl" scale="1 1 1"/>
+        <mesh filename="package://pcr_description/meshes/module_cart.stl" scale="1 1 1"/>
       </geometry>
       <origin xyz="0 0 0" rpy="0 0 0"/>
@@ -82,5 +82,5 @@
       <origin xyz="0 0 0" rpy="0 0 0"/>
       <geometry>
-        <mesh filename="package://pf400_description/meshes/module_cart.stl" scale="1 1 1"/>
+        <mesh filename="package://pcr_description/meshes/module_cart.stl" scale="1 1 1"/>
       </geometry>
       <material name="darkbluegreen"/>
@@ -88,5 +88,5 @@
     <collision>
       <geometry>
-        <mesh filename="package://pf400_description/meshes/module_cart.stl" scale="1 1 1"/>
+        <mesh filename="package://pcr_description/meshes/module_cart.stl" scale="1 1 1"/>
       </geometry>
       <origin xyz="0 0 0" rpy="0 0 0"/>
@@ -97,5 +97,5 @@
       <origin xyz="0 0 0" rpy="0 0 0"/>
       <geometry>
-        <mesh filename="package://pf400_description/meshes/module_cart.stl" scale="1 1 1"/>
+        <mesh filename="package://pcr_description/meshes/module_cart.stl" scale="1 1 1"/>
       </geometry>
       <material name="darkbluegreen"/>
@@ -103,5 +103,5 @@
     <collision>
       <geometry>
-        <mesh filename="package://pf400_description/meshes/module_cart.stl" scale="1 1 1"/>
+        <mesh filename="package://pcr_description/meshes/module_cart.stl" scale="1 1 1"/>
       </geometry>
       <origin xyz="0 0 0" rpy="0 0 0"/>
@@ -112,5 +112,5 @@
       <origin xyz="0 0 0" rpy="0 0 0"/>
       <geometry>
-        <mesh filename="package://pf400_description/meshes/module_cart.stl" scale="1 1 1"/>
+        <mesh filename="package://pcr_description/meshes/module_cart.stl" scale="1 1 1"/>
       </geometry>
       <material name="darkbluegreen"/>
@@ -118,5 +118,5 @@
     <collision>
       <geometry>
-        <mesh filename="package://pf400_description/meshes/module_cart.stl" scale="1 1 1"/>
+        <mesh filename="package://pcr_description/meshes/module_cart.stl" scale="1 1 1"/>
       </geometry>
       <origin xyz="0 0 0" rpy="0 0 0"/>
@@ -125,7 +125,7 @@
   <link name="${prefix}pf400_cart">
     <visual>
-      <origin xyz="-1.592 0.2605 -0.015" rpy="1.5708 0 0"/>
+      <origin xyz="-1.592 0.2605 -0.0" rpy="1.5708 0 0"/>
       <geometry>
-        <mesh filename="package://pf400_description/meshes/pf400_table.STL" scale="0.001 0.001 0.001"/>
+        <mesh filename="package://pcr_description/meshes/pf400_table.STL" scale="0.001 0.001 0.001"/>
       </geometry>
       <material name="darkbluegreen"/>
@@ -133,7 +133,7 @@
     <collision>
       <geometry>
-        <mesh filename="package://pf400_description/meshes/pf400_table.STL" scale="0.001 0.001 0.001"/>
+        <mesh filename="package://pcr_description/meshes/pf400_table.STL" scale="0.001 0.001 0.001"/>
       </geometry>
-      <origin xyz="-1.592 0.261 -0.015" rpy="1.5708 0 0"/>
+      <origin xyz="-1.592 0.261 -0.0" rpy="1.5708 0 0"/>
     </collision>
   </link>
@@ -143,5 +143,5 @@
     <child link="${prefix}cart_1"/>
     <axis xyz="0 0 1"/>
-    <origin xyz="1.0 0.83 0" rpy="0 0 0"/>
+    <origin xyz="1.0 0.91 0.005" rpy="0 0 0"/>
     <limit effort="1000.0" lower="0" upper="0" velocity="0.5"/>
   </joint>
@@ -150,5 +150,5 @@
     <child link="${prefix}cart_2"/>
     <axis xyz="0 0 1"/>
-    <origin xyz="0.25 0.83 0" rpy="0 0 0"/>
+    <origin xyz="0.25 0.91 0.005" rpy="0 0 0"/>
     <limit effort="1000.0" lower="0" upper="0" velocity="0.5"/>
   </joint>
@@ -157,5 +157,5 @@
     <child link="${prefix}cart_3"/>
     <axis xyz="0 0 1"/>
-    <origin xyz="-0.50 0.83  0" rpy="0 0 0"/>
+    <origin xyz="-0.50 0.91  0.005" rpy="0 0 0"/>
     <limit effort="1000.0" lower="0" upper="0" velocity="0.5"/>
   </joint>
@@ -164,5 +164,5 @@
     <child link="${prefix}cart_4"/>
     <axis xyz="0 0 1"/>
-    <origin xyz="-1.25 0.83  0" rpy="0 0 0"/>
+    <origin xyz="-1.25 0.91  0.005" rpy="0 0 0"/>
     <limit effort="1000.0" lower="0" upper="0" velocity="0.5"/>
   </joint>
@@ -171,5 +171,5 @@
     <child link="${prefix}cart_5"/>
     <axis xyz="0 0 1"/>
-    <origin xyz="1.00 -0.46 0" rpy="0 0 0"/>
+    <origin xyz="1.00 -0.54 0.005" rpy="0 0 0"/>
     <limit effort="1000.0" lower="0" upper="0" velocity="0.5"/>
   </joint>
@@ -178,5 +178,5 @@
     <child link="${prefix}cart_6"/>
     <axis xyz="0 0 1"/>
-    <origin xyz="0.25 -0.46 0" rpy="0 0 0"/>
+    <origin xyz="0.25 -0.54 0.005" rpy="0 0 0"/>
     <limit effort="1000.0" lower="0" upper="0" velocity="0.5"/>
   </joint>
@@ -185,5 +185,5 @@
     <child link="${prefix}cart_7"/>
     <axis xyz="0 0 1"/>
-    <origin xyz="-0.50 -0.46 0" rpy="0 0 0"/>
+    <origin xyz="-0.50 -0.54 0.005" rpy="0 0 0"/>
     <limit effort="1000.0" lower="0" upper="0" velocity="0.5"/>
   </joint>
@@ -192,5 +192,5 @@
     <child link="${prefix}cart_8"/>
     <axis xyz="0 0 1"/>
-    <origin xyz="-1.25 -0.46 0" rpy="0 0 0"/>
+    <origin xyz="-1.25 -0.54 0.005" rpy="0 0 0"/>
     <limit effort="1000.0" lower="0" upper="0" velocity="0.5"/>
   </joint>

Commit message: Clean up

File: pcr_description/urdf/module_carts.urdf.xacro (robot description, xacro)
@@ -180,5 +180,5 @@
     <origin xyz="0.25 -0.54 0.005" rpy="0 0 0"/>
     <limit effort="1000.0" lower="0" upper="0" velocity="0.5"/>
-  </joint>
+  </joint>y
   <joint name="pf400_cart_to_cart_7" type="fixed">
     <parent link="${prefix}pf400_cart"/>
